Commit message: 0424

File: a1_description/urdf/a1_kinova.urdf (robot description, URDF)
Before this commit: robot a1, 23 links, 22 joints
Links:
- added link j2s6s200_end_effector, mass 0.0
- added link j2s6s200_link_1, mass 0.7477; collision mesh filename=package://kinova_description/meshes/shoulder.dae; visual mesh filename=package://kinova_description/meshes/ring_big.dae
- added link j2s6s200_link_2, mass 0.99; collision mesh filename=package://kinova_description/meshes/arm.dae; visual mesh filename=package://kinova_description/meshes/arm.dae
- added link j2s6s200_link_3, mass 0.6763; collision mesh filename=package://kinova_description/meshes/forearm.dae; visual mesh filename=package://kinova_description/meshes/forearm.dae
- added link j2s6s200_link_4, mass 0.463; collision mesh filename=package://kinova_description/meshes/wrist_spherical_1.dae; visual mesh filename=package://kinova_description/meshes/ring_small.dae
- added link j2s6s200_link_5, mass 0.463; collision mesh filename=package://kinova_description/meshes/wrist_spherical_2.dae; visual mesh filename=package://kinova_description/meshes/ring_small.dae
- added link j2s6s200_link_6, mass 0.99; collision mesh filename=package://kinova_description/meshes/hand_2finger.dae; visual mesh filename=package://kinova_description/meshes/hand_2finger.dae
- added link j2s6s200_link_base, mass 0.46784; collision mesh filename=package://kinova_description/meshes/base.dae; visual mesh filename=package://kinova_description/meshes/base.dae
- added link j2s6s200_link_finger_1, mass 0.01; collision mesh filename=package://kinova_description/meshes/finger_proximal.dae; visual mesh filename=package://kinova_description/meshes/finger_proximal.dae
- added link j2s6s200_link_finger_2, mass 0.01; collision mesh filename=package://kinova_description/meshes/finger_proximal.dae; visual mesh filename=package://kinova_description/meshes/finger_proximal.dae
- added link j2s6s200_link_finger_tip_1, mass 0.01; collision mesh filename=package://kinova_description/meshes/finger_distal.dae; visual mesh filename=package://kinova_description/meshes/finger_distal.dae
- added link j2s6s200_link_finger_tip_2, mass 0.01; collision mesh filename=package://kinova_description/meshes/finger_distal.dae; visual mesh filename=package://kinova_description/meshes/finger_distal.dae
Joints:
- added joint j2s6s200_joint_1: type revolute, parent j2s6s200_link_base, child j2s6s200_link_1, origin xyz=0 0 0.15675 rpy=0 3.14159265359 0, axis 0 0 1, limit lower=-6.28318530718 upper=6.28318530718 effort=40 velocity=0.628318530718
- added joint j2s6s200_joint_2: type revolute, parent j2s6s200_link_1, child j2s6s200_link_2, origin xyz=0 0.0016 -0.11875 rpy=-1.57079632679 0 3.14159265359, axis 0 0 1, limit lower=0.820304748437 upper=5.46288055874 effort=80 velocity=0.628318530718
- added joint j2s6s200_joint_3: type revolute, parent j2s6s200_link_2, child j2s6s200_link_3, origin xyz=0 -0.410 0 rpy=0 3.14159265359 0, axis 0 0 1, limit lower=0.331612557879 upper=5.9515727493 effort=40 velocity=0.628318530718
- added joint j2s6s200_joint_4: type revolute, parent j2s6s200_link_3, child j2s6s200_link_4, origin xyz=0 0.2073 -0.0114 rpy=-1.57079632679 0 3.14159265359, axis 0 0 1, limit lower=-6.28318530718 upper=6.28318530718 effort=20 velocity=0.837758040957
- added joint j2s6s200_joint_5: type revolute, parent j2s6s200_link_4, child j2s6s200_link_5, origin xyz=0 0 -0.10375 rpy=1.57079632679 0 3.14159265359, axis 0 0 1, limit lower=0.523598775598 upper=5.75958653158 effort=20 velocity=0.837758040957
- added joint j2s6s200_joint_6: type revolute, parent j2s6s200_link_5, child j2s6s200_link_6, origin xyz=0 0.10375 0 rpy=-1.57079632679 0 3.14159265359, axis 0 0 1, limit lower=-6.28318530718 upper=6.28318530718 effort=20 velocity=0.837758040957
- added joint j2s6s200_joint_end_effector: type fixed, parent j2s6s200_link_6, child j2s6s200_end_effector, origin xyz=0 0 -0.1600 rpy=3.14159265359 1.57079632679 0, axis 0 0 0, limit lower=0 upper=0 effort=2000 velocity=1
- added joint j2s6s200_joint_finger_1: type fixed, parent j2s6s200_link_6, child j2s6s200_link_finger_1, origin xyz=-0.0025 0.03095 -0.11482 rpy=-1.570796327 .649262481663582 1.57079632679490, axis 0 0 1, limit lower=0 upper=1.51 effort=2 velocity=1
- added joint j2s6s200_joint_finger_2: type fixed, parent j2s6s200_link_6, child j2s6s200_link_finger_2, origin xyz=-0.0025 -0.03095 -0.11482 rpy=-1.570796327 .649262481663582 -1.57079632679490, axis 0 0 1, limit lower=0 upper=1.51 effort=2 velocity=1
- added joint j2s6s200_joint_finger_tip_1: type fixed, parent j2s6s200_link_finger_1, child j2s6s200_link_finger_tip_1, origin xyz=0.044 -0.003 0 rpy=0 0 0, axis 0 0 1, limit lower=0 upper=2 effort=2 velocity=1
- added joint j2s6s200_joint_finger_tip_2: type fixed, parent j2s6s200_link_finger_2, child j2s6s200_link_finger_tip_2, origin xyz=0.044 -0.003 0 rpy=0 0 0, axis 0 0 1, limit lower=0 upper=2 effort=2 velocity=1
- added joint jaco_mounting_block_to_j2s6s200_link_base: type fixed, parent trunk, child j2s6s200_link_base, origin xyz=0.000 0.000 0.000 rpy=0 0 1.57079632679, axis 0 0 0, limit lower=0 upper=0 effort=0 velocity=0
